Commit message: adefbec

File: src/motor_controller/gazebo_models/carModelURDF.urdf (robot description, URDF)
Before this commit: robot simple_robot, 3 links, 2 joints
Links:
- added link rear_left_wheel_link, mass 0.2; collision cylinder length=0.05 radius=0.1; visual cylinder length=0.05 radius=0.1
- added link rear_right_wheel_link, mass 0.2; collision cylinder length=0.05 radius=0.1; visual cylinder length=0.05 radius=0.1
Joints:
- removed joint left_wheel_joint
- removed joint right_wheel_joint
- added joint front_left_wheel_joint: type revolute, parent base_link, child front_left_wheel_link, origin xyz=0.25 0.15 0, axis 0 1 0, limit effort=50 velocity=10
- added joint front_right_wheel_joint: type revolute, parent base_link, child front_right_wheel_link, origin xyz=0.25 -0.15 0, axis 0 1 0, limit effort=50 velocity=10
- added joint rear_left_wheel_joint: type revolute, parent base_link, child rear_left_wheel_link, origin xyz=-0.25 0.15 0, axis 0 1 0, limit effort=50 velocity=10
- added joint rear_right_wheel_joint: type revolute, parent base_link, child rear_right_wheel_link, origin xyz=-0.25 -0.15 0, axis 0 1 0, limit effort=50 velocity=10
