Commit message: fixed the ros control setup, final issue is launching, also manual launch of teleops keyboard required

File: install/motor_controller/share/motor_controller/gazebo_models/carModelURDF.urdf (robot description, URDF)
Before this commit: robot four_wheel_drive_robot, 5 links, 4 joints
Links:
- removed link left_wheel_link
- removed link rear_left_wheel_link
- removed link rear_right_wheel_link
- removed link right_wheel_link
- added link front_left_wheel, mass 0.1; collision cylinder length=0.05 radius=0.1; visual cylinder length=0.05 radius=0.1
- added link front_right_wheel, mass 0.1; collision cylinder length=0.05 radius=0.1; visual cylinder length=0.05 radius=0.1
- added link rear_left_wheel, mass 0.1; collision cylinder length=0.05 radius=0.1; visual cylinder length=0.05 radius=0.1
- added link rear_right_wheel, mass 0.1; collision cylinder length=0.05 radius=0.1; visual cylinder length=0.05 radius=0.1
- link base_link: geometry 
Joints:
- joint front_left_wheel_joint: child front_left_wheel_link -> front_left_wheel; limit effort=50 velocity=10 -> lower=-1.57 upper=1.57 effort=100 velocity=10; origin xyz=0.25 0.15 0 -> xyz=-0.25 0.25 0 rpy=0 0 0
- joint front_right_wheel_joint: child front_right_wheel_link -> front_right_wheel; limit effort=50 velocity=10 -> lower=-1.57 upper=1.57 effort=100 velocity=10; origin xyz=0.25 -0.15 0 -> xyz=-0.25 -0.25 0 rpy=0 0 0
- joint rear_left_wheel_joint: axis 0 1 0 -> (none); child rear_left_wheel_link -> rear_left_wheel; limit effort=50 velocity=10 -> (none); origin xyz=-0.25 0.15 0 -> xyz=0.25 0.25 0 rpy=0 0 0; type revolute -> fixed
- joint rear_right_wheel_joint: axis 0 1 0 -> (none); child rear_right_wheel_link -> rear_right_wheel; limit effort=50 velocity=10 -> (none); origin xyz=-0.25 -0.15 0 -> xyz=0.25 -0.25 0 rpy=0 0 0; type revolute -> fixed

Commit message: working code, minus controller

File: install/motor_controller/share/motor_controller/gazebo_models/carModelURDF.urdf (robot description, URDF)
Before this commit: robot four_wheeled_car, 5 links, 4 joints
Links:
- link base_link: mass 1.0 -> 10; geometry collision box size=1.0 0.5 0.2; visual box size=1.0 0.5 0.2
- link front_left_wheel: mass 0.1 -> 1; geometry collision cylinder length=0.05 radius=0.15; visual cylinder length=0.05 radius=0.15
- link front_right_wheel: mass 0.1 -> 1; geometry collision cylinder length=0.05 radius=0.15; visual cylinder length=0.05 radius=0.15
- link rear_left_wheel: mass 0.1 -> 1; geometry collision cylinder length=0.05 radius=0.15; visual cylinder length=0.05 radius=0.15
- link rear_right_wheel: mass 0.1 -> 1; geometry collision cylinder length=0.05 radius=0.15; visual cylinder length=0.05 radius=0.15
Joints:
- joint front_left_wheel_joint: axis 0 1 0 -> 0 0 1; limit lower=-1.57 upper=1.57 effort=100 velocity=10 -> (none); origin xyz=-0.25 0.25 0 rpy=0 0 0 -> xyz=0.5 0.275 0.1 rpy=${pi/2} 0 0; type revolute -> continuous
- joint front_right_wheel_joint: axis 0 1 0 -> 0 0 1; limit lower=-1.57 upper=1.57 effort=100 velocity=10 -> (none); origin xyz=-0.25 -0.25 0 rpy=0 0 0 -> xyz=0.5 -0.275 0.1 rpy=-${pi/2} 0 0; type revolute -> continuous
- joint rear_left_wheel_joint: axis (none) -> 0 0 1; origin xyz=0.25 0.25 0 rpy=0 0 0 -> xyz=-0.5 0.275 0.1 rpy=${pi/2} 0 0; type fixed -> continuous
- joint rear_right_wheel_joint: axis (none) -> 0 0 1; origin xyz=0.25 -0.25 0 rpy=0 0 0 -> xyz=-0.5 -0.275 0.1 rpy=-${pi/2} 0 0; type fixed -> continuous
