Commit message: another trial and getting the launch to work

File: install/motor_controller/share/motor_controller/gazebo_models/carModelURDF.urdf.xacro (robot description, xacro)
@@ -65,5 +65,5 @@
   </joint>
   <!-- Rear Left Wheel Joint -->
-  <joint name=left_wheel_joint" type="revolute">
+  <joint name="left_wheel_joint" type="revolute">
     <parent link="car_body"/>
     <child link="rear_left_wheel"/>
@@ -73,5 +73,5 @@
   </joint>
   <!-- Rear Right Wheel Joint -->
-  <joint name=right_wheel_joint" type="revolute">
+  <joint name="right_wheel_joint" type="revolute">
     <parent link="car_body"/>
     <child link="rear_right_wheel"/>

Commit message: same issue but little better

File: install/motor_controller/share/motor_controller/gazebo_models/carModelURDF.urdf.xacro (robot description, xacro)
@@ -183,7 +183,7 @@
     <gazebo>
         <plugin name="gazebo_ros2_control" filename="libgazebo_ros2_control.so">
-            <parameters>$(find motor_controller)/config/controllers.yaml</parameters>
+            <parameters>$(find motor_controller)/gazebo_models/controller.yaml</parameters>
         </plugin>
-    </gazebo>
+</gazebo>
     <!-- Base color in Gazebo -->
     <gazebo reference="base_link">

File: src/motor_controller/gazebo_models/carModelURDF.urdf.xacro (robot description, xacro)
@@ -4,5 +4,5 @@
     <xacro:arg name="prefix" default=""/>
     <!-- Define materials -->
-    <material name="blue">
+    <material name="red">
         <color rgba="0 0 1 1"/>
     </material>
@@ -183,5 +183,5 @@
     <gazebo>
         <plugin name="gazebo_ros2_control" filename="libgazebo_ros2_control.so">
-            <parameters>$(find motor_controller)/config/controllers.yaml</parameters>
+            <parameters>$(find motor_controller)/gazebo_models/controller.yaml</parameters>
         </plugin>
     </gazebo>

Commit message: Controller fixed, now deal with topics for correctly addressing inputs

File: install/motor_controller/share/motor_controller/gazebo_models/carModelURDF.urdf.xacro (robot description, xacro)
@@ -4,5 +4,5 @@
     <xacro:arg name="prefix" default=""/>
     <!-- Define materials -->
-    <material name="blue">
+    <material name="red">
         <color rgba="0 0 1 1"/>
     </material>
@@ -141,5 +141,4 @@
         <axis xyz="0 0 1"/>
     </joint>
-    <!-- Rest of the file remains the same -->
     <!-- ros2_control section -->
     <ros2_control name="GazeboSystem" type="system">
@@ -185,8 +184,8 @@
             <parameters>$(find motor_controller)/gazebo_models/controller.yaml</parameters>
         </plugin>
-</gazebo>
+    </gazebo>
     <!-- Base color in Gazebo -->
     <gazebo reference="base_link">
-        <material>Gazebo/Blue</material>
+        <material>Gazebo/Red</material>
     </gazebo>
 </robot>

File: src/motor_controller/gazebo_models/carModelURDF.urdf.xacro (robot description, xacro)
@@ -141,5 +141,4 @@
         <axis xyz="0 0 1"/>
     </joint>
-    <!-- Rest of the file remains the same -->
     <!-- ros2_control section -->
     <ros2_control name="GazeboSystem" type="system">
@@ -188,5 +187,5 @@
     <!-- Base color in Gazebo -->
     <gazebo reference="base_link">
-        <material>Gazebo/Blue</material>
+        <material>Gazebo/Red</material>
     </gazebo>
 </robot>
